Commit message: working sample gazebo viewer

File: mhsboat/urdf/tuppy.urdf (robot description, URDF)
Before this commit: robot tuppy, 0 links, 0 joints
Links:
- added link base_link; collision box size=0.4 0.25 0.1; visual box size=0.4 0.25 0.1
- added link center_cross_beam; collision box size=0.025 0.5 0.025; visual box size=0.025 0.5 0.025
- added link front_cross_beam; collision box size=0.025 0.5 0.025; visual box size=0.025 0.5 0.025
- added link imu_link; collision box size=0.025 0.025 0.025; visual box size=0.025 0.025 0.025
- added link left_float; collision box size=0.8 0.15 0.15; visual box size=0.8 0.15 0.15
- added link left_propeller; visual cylinder length=0.025 radius=0.05
- added link lidar_link; collision cylinder length=0.07 radius=0.05; visual cylinder length=0.07 radius=0.05
- added link rear_cross_beam; collision box size=0.025 0.5 0.025; visual box size=0.025 0.5 0.025
- added link right_float; collision box size=0.8 0.15 0.15; visual box size=0.8 0.15 0.15
- added link right_propeller; visual cylinder length=0.025 radius=0.05
Joints:
- added joint center_cross_bream_joint: type fixed, parent base_link, child center_cross_beam, origin xyz=0.15 0.0 -0.0625
- added joint front_cross_bream_joint: type fixed, parent base_link, child front_cross_beam, origin xyz=0.35 0.0 -0.0625
- added joint imu_joint: type fixed, parent base_link, child imu_link, origin xyz=0.15 0 0
- added joint left_float_joint: type fixed, parent base_link, child left_float, origin xyz=0.15 0.25 -0.15
- added joint left_prop_joint: type continuous, parent base_link, child left_propeller, origin xyz=-0.3 0.25 -0.25 rpy=0 ${pi/2} 0, axis 0 0 1
- added joint lidar_joint: type fixed, parent base_link, child lidar_link, origin xyz=0.35 0.0 -0.015
- added joint rear_cross_bream_joint: type fixed, parent base_link, child rear_cross_beam, origin xyz=-0.15 0.0 -0.0625
- added joint right_float_joint: type fixed, parent base_link, child right_float, origin xyz=0.15 -0.25 -0.15
- added joint right_prop_joint: type continuous, parent base_link, child right_propeller, origin xyz=-0.3 -0.25 -0.25 rpy=0 ${pi/2} 0, axis 0 0 1

Commit message: added velodyne sensor integration and robot localization node; updated dependencies and rviz configuration

File: mhsboat/urdf/tuppy.urdf (robot description, URDF)
Before this commit: robot tuppy, 10 links, 9 joints
Links:
- removed link lidar_link
Joints:
- removed joint lidar_joint

Commit message: Revert "added velodyne sensor integration and robot localization node; updated dependencies and rviz configuration"
This reverts commit 44a7079acbed08911b938ed2682c045dbca0f684.

File: mhsboat/urdf/tuppy.urdf (robot description, URDF)
Before this commit: robot tuppy, 9 links, 8 joints
Links:
- added link lidar_link; collision cylinder length=0.07 radius=0.05; visual cylinder length=0.07 radius=0.05
Joints:
- added joint lidar_joint: type fixed, parent base_link, child lidar_link, origin xyz=0.35 0.0 -0.015
